File: Ari-First-PCB/Ari-First-PCB.kicad_sch (KiCad schematic)
At the start: 10 parts, among them Q1 Q_NPN_BCE, Q2 Q_NPN_BCE

Commit message: Add files via upload
Parts:
- BT1: value 3 -> CR2032 (3V)
- D1, D2: value LED -> LED 5mm
- Q1, Q2: value Q_NPN_BCE -> 2N3904 transistor
- R1: value R_Photo -> Photoresistor (LDR)
- R10: value 47k -> 47kΩ
- R11: value 4.7k -> 4.7kΩ
- R2, R3: value 470 -> 470Ω
Changed lines of the file:
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@@
 			)
 		)
-		(property "Value" "470"
+		(property "Value" "470Ω"
 			(at 210.82 86.3599 0)
 			(show_name no)
@@
 			)
 		)
-		(property "Value" "LED"
+		(property "Value" "LED 5mm"
 			(at 224.4725 93.98 0)
 			(show_name no)
@@
 			)
 		)
-		(property "Value" "Q_NPN_BCE"
+		(property "Value" "2N3904 transistor"
 			(at 231.14 142.2399 0)
 			(show_name no)
@@
 			)
 		)
-		(property "Value" "3"
+		(property "Value" "CR2032 (3V)"
 			(at 170.18 85.7884 0)
 			(show_name no)
@@
 			)
 		)
-		(property "Value" "470"
+		(property "Value" "470Ω"
 			(at 227.33 86.3599 0)
 			(show_name no)
@@
 			)
 		)
-		(property "Value" "LED"
+		(property "Value" "LED 5mm"
 			(at 207.9625 93.98 0)
 			(show_name no)
@@
 			)
 		)
-		(property "Value" "Q_NPN_BCE"
+		(property "Value" "2N3904 transistor"
 			(at 207.01 126.9999 0)
 			(show_name no)
@@
 			)
 		)
-		(property "Value" "4.7k"
+		(property "Value" "4.7kΩ"
 			(at 191.77 123.1899 0)
 			(show_name no)
@@
 			)
 		)
-		(property "Value" "R_Photo"
+		(property "Value" "Photoresistor (LDR)"
 			(at 229.87 126.9999 0)
 			(show_name no)
@@
 			)
 		)
-		(property "Value" "47k"
+		(property "Value" "47kΩ"
 			(at 217.17 138.4299 0)
 			(show_name no)
